Commit message: Correct body-coxa servos to MG996R and record stair retraining

File: isaaclab_project/assets/spiderbot_variants/onshape_20260928/robot.training.urdf (robot description, URDF)
Before this commit: robot dksh_onshape_hexapod_20260928, 25 links, 24 joints
Joints:
- joint leg_0_hip_joint: limit lower=-1.5707963267948966 upper=1.5707963267948966 effort=0.13239000 velocity=10.47197551 -> lower=-1.5707963267948966 upper=1.5707963267948966 effort=0.69136883 velocity=5.51156606
- joint leg_1_hip_joint: limit lower=-1.5707963267948966 upper=1.5707963267948966 effort=0.13239000 velocity=10.47197551 -> lower=-1.5707963267948966 upper=1.5707963267948966 effort=0.69136883 velocity=5.51156606
- joint leg_2_hip_joint: limit lower=-1.5707963267948966 upper=1.5707963267948966 effort=0.13239000 velocity=10.47197551 -> lower=-1.5707963267948966 upper=1.5707963267948966 effort=0.69136883 velocity=5.51156606
- joint leg_3_hip_joint: limit lower=-1.5707963267948966 upper=1.5707963267948966 effort=0.13239000 velocity=10.47197551 -> lower=-1.5707963267948966 upper=1.5707963267948966 effort=0.69136883 velocity=5.51156606
- joint leg_4_hip_joint: limit lower=-1.5707963267948966 upper=1.5707963267948966 effort=0.13239000 velocity=10.47197551 -> lower=-1.5707963267948966 upper=1.5707963267948966 effort=0.69136883 velocity=5.51156606
- joint leg_5_hip_joint: limit lower=-1.5707963267948966 upper=1.5707963267948966 effort=0.13239000 velocity=10.47197551 -> lower=-1.5707963267948966 upper=1.5707963267948966 effort=0.69136883 velocity=5.51156606
